Commit message: first commit

File: test.urdf (robot description, URDF)
Before this commit: robot spot, 24 links, 23 joints
Links:
- added link base_inertia, mass 0.6; collision box size=0.114 0.2 0.1; visual mesh filename=package://mini_ros/stl/OpenQuadruped/MAINBODY.stl scale=1 1 1
- link base_link: mass 0.6 -> None; geometry 
- link front_left_lower_leg: geometry collision box size=0.035 0.035 0.12; visual mesh filename=package://mini_ros/stl/OpenQuadruped/LEFT_LOWER_LEG.stl scale=1 1 1
Joints:
- added joint base_base: type fixed, parent base_link, child base_inertia, origin xyz=0 0 0 rpy=0 0 0
- joint motor_back_left_hip: limit lower=-1.04 upper=1.04 effort=1000.0 velocity=0.7 -> lower=-1.04 upper=1.04 effort=4.0 velocity=4.0; origin xyz=-0.1365 0.0394 0.022 rpy=0 0 0 -> xyz=-0.1365 0.039400000000000004 0.022000000000000006 rpy=0 0 0
- joint motor_back_left_lower_leg: limit lower=-2.9 upper=1.57079632679 effort=1000.0 velocity=0.7 -> lower=-2.9 upper=1.5707963267948966 effort=4.0 velocity=4.0
- joint motor_back_left_upper_leg: limit lower=-1.57079632679 upper=2.59 effort=1000.0 velocity=0.7 -> lower=-1.5707963267948966 upper=2.59 effort=4.0 velocity=4.0
- joint motor_back_right_hip: limit lower=-1.04 upper=1.04 effort=1000.0 velocity=0.7 -> lower=-1.04 upper=1.04 effort=4.0 velocity=4.0; origin xyz=-0.1365 -0.0394 0.022 rpy=0 0 0 -> xyz=-0.1365 -0.039400000000000004 0.022000000000000006 rpy=0 0 0
- joint motor_back_right_lower_leg: limit lower=-2.9 upper=1.57079632679 effort=1000.0 velocity=0.7 -> lower=-2.9 upper=1.5707963267948966 effort=4.0 velocity=4.0
- joint motor_back_right_upper_leg: limit lower=-1.57079632679 upper=2.59 effort=1000.0 velocity=0.7 -> lower=-1.5707963267948966 upper=2.59 effort=4.0 velocity=4.0
- joint motor_front_left_hip: limit lower=-1.04 upper=1.04 effort=1000.0 velocity=0.7 -> lower=-1.04 upper=1.04 effort=4.0 velocity=4.0; origin xyz=0.0915 0.0394 0.022 rpy=0 0 0 -> xyz=0.0915 0.039400000000000004 0.022000000000000006 rpy=0 0 0
- joint motor_front_left_lower_leg: limit lower=-2.9 upper=1.57079632679 effort=1000.0 velocity=0.7 -> lower=-2.9 upper=1.5707963267948966 effort=4.0 velocity=4.0
- joint motor_front_left_upper_leg: limit lower=-1.57079632679 upper=2.59 effort=1000.0 velocity=0.7 -> lower=-1.5707963267948966 upper=2.59 effort=4.0 velocity=4.0
- joint motor_front_right_hip: limit lower=-1.04 upper=1.04 effort=1000.0 velocity=0.7 -> lower=-1.04 upper=1.04 effort=4.0 velocity=4.0; origin xyz=0.0915 -0.0394 0.022 rpy=0 0 0 -> xyz=0.0915 -0.039400000000000004 0.022000000000000006 rpy=0 0 0
- joint motor_front_right_lower_leg: limit lower=-2.9 upper=1.57079632679 effort=1000.0 velocity=0.7 -> lower=-2.9 upper=1.5707963267948966 effort=4.0 velocity=4.0
- joint motor_front_right_upper_leg: limit lower=-1.57079632679 upper=2.59 effort=1000.0 velocity=0.7 -> lower=-1.5707963267948966 upper=2.59 effort=4.0 velocity=4.0
